Commit message: fix(topics): odom -> odom_combined

File: src/turn_on_rai_robot/urdf/mini_mec_gazebo.urdf.xacro (robot description, xacro)
@@ -52,6 +52,6 @@
   <xacro:wheel name="rf" x="0.079" y="-0.099" />
   <xacro:wheel name="rb" x="-0.079" y="-0.099" />
-  <link name="laser_link"><visual><geometry><cylinder radius="0.025" length="0.03" /></geometry></visual></link>
-  <joint name="laser_joint" type="fixed"><origin xyz="0.03 0 0.14"/><parent link="base_link"/><child link="laser_link"/></joint>
+  <link name="laser"><visual><geometry><cylinder radius="0.025" length="0.03" /></geometry></visual></link>
+  <joint name="laser_joint" type="fixed"><origin xyz="0.03 0 0.14"/><parent link="base_link"/><child link="laser"/></joint>
   <link name="camera_link"><visual><geometry><box size="0.035 0.05 0.025" /></geometry></visual></link>
   <joint name="camera_joint" type="fixed"><origin xyz="0.105 0 0.10"/><parent link="base_link"/><child link="camera_link"/></joint>
@@ -82,9 +82,9 @@
         <command_topic>cmd_vel</command_topic>
         <publish_odom>true</publish_odom>
-        <publish_odom_tf>true</publish_odom_tf>
+        <publish_odom_tf>false</publish_odom_tf>
         <publish_wheel_tf>false</publish_wheel_tf>
-        <odometry_topic>odom_combined</odometry_topic>
-        <odometry_frame>odom_combined</odometry_frame>
-        <robot_base_frame>base_link</robot_base_frame>
+        <odometry_topic>odom</odometry_topic>
+        <odometry_frame>odom</odometry_frame>
+        <robot_base_frame>base_footprint</robot_base_frame>
       </plugin>
     </gazebo>
@@ -99,8 +99,8 @@
         <command_topic>cmd_vel</command_topic>
         <publish_odom>true</publish_odom>
-        <publish_odom_tf>true</publish_odom_tf>
-        <odometry_topic>odom_combined</odometry_topic>
-        <odometry_frame>odom_combined</odometry_frame>
-        <robot_base_frame>base_link</robot_base_frame>
+        <publish_odom_tf>false</publish_odom_tf>
+        <odometry_topic>odom</odometry_topic>
+        <odometry_frame>odom</odometry_frame>
+        <robot_base_frame>base_footprint</robot_base_frame>
         <covariance_x>0.0001</covariance_x>
         <covariance_y>0.0001</covariance_y>
@@ -110,5 +110,5 @@
   </xacro:if>
   <!-- Lidar sensor plugin -->
-  <gazebo reference="laser_link">
+  <gazebo reference="laser">
     <sensor type="ray" name="laser_sensor">
       <pose>0 0 0 0 0 0</pose>
@@ -140,5 +140,5 @@
         </ros>
         <output_type>sensor_msgs/LaserScan</output_type>
-        <frame_name>laser_link</frame_name>
+        <frame_name>laser</frame_name>
       </plugin>
     </sensor>
