Commit message: fix(topics): odom vs base_link

File: src/rai_robot_urdf/rai_robot_urdf/urdf/mini_mec_robot.urdf (robot description, URDF)
Before this commit: robot mini_mec_robot, 8 links, 7 joints
Joints:
- joint camera_joint: origin xyz=0.10709468678297 0.000317092708037946 0.076204 rpy=0 0 0 -> xyz=0.10709468678297 0.000317092708037946 0.21 rpy=0 -0.34906585 0

File: src/turn_on_rai_robot/urdf/mini_mec_gazebo.urdf.xacro (robot description, xacro)
@@ -55,5 +55,5 @@
   <joint name="laser_joint" type="fixed"><origin xyz="0.03 0 0.14"/><parent link="base_link"/><child link="laser"/></joint>
   <link name="camera_link"><visual><geometry><box size="0.035 0.05 0.025" /></geometry></visual></link>
-  <joint name="camera_joint" type="fixed"><origin xyz="0.105 0 0.10"/><parent link="base_link"/><child link="camera_link"/></joint>
+  <joint name="camera_joint" type="fixed"><origin xyz="0.105 0 0.21" rpy="0 -0.34906585 0"/><parent link="base_link"/><child link="camera_link"/></joint>
   <!-- ROS optical-frame convention (docs/config camera_optical_frame):
        body camera_link (x-forward) -> optical (x-right, y-down, z-forward).
